File: DC-AC-Inverter-EGS-1.0.1/DC-AC-Inverter-EGS.kicad_pcb (KiCad board)
At the start: 2 copper layers, 90 x 44 mm, 46 parts, among them J1 Fan, J2 EGS002 MODULE, J4 TR/IN, J5 AC/OUT, J6 DC IN, Q1 RM10N100LDV-T, Q2 S8050, Q3 IRF3205, Q4 IRF3205, Q5 IRF3205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

Commit message: Update
Other:
- board text removed: "VS1"
- board text removed: "VS2"
Changed lines of the file:
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@@
 			(drillshape 0)
 			(scaleselection 1)
-			(outputdirectory "DC-AC-Inverter-EG-Gerber/")
+			(outputdirectory "DC-AC-Inverter-EGS-Gerber/")
 		)
 	)
@@
 		)
 	)
-	(gr_text "VS2"
-		(at 141.605 93.757905 -90)
+	(gr_text "TR1"
+		(at 141.605 93.757905 270)
 		(layer "B.SilkS")
 		(effects
@@
 		)
 	)
-	(gr_text "VS1"
-		(at 131.445 93.757905 -90)
+	(gr_text "TR2"
+		(at 131.445 93.757905 270)
 		(layer "B.SilkS")
 		(effects
