File: DC-AC-Inverter-EGS-1.0.1/DC-AC-Inverter-EGS.kicad_pcb (KiCad board)
At the start: 2 copper layers, 90 x 44 mm, 46 parts, among them J1 Fan, J2 EGS002 MODULE, J4 TR/IN, J5 AC/OUT, J6 DC IN, Q1 RM10N100LDV-T, Q2 S8050, Q3 IRF3205, Q4 IRF3205, Q5 IRF3205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

Commit message: Update 1.0.2
Parts:
- C4: value 22uF 10V -> 47uF 10V
Connections:
- C7 pad 2: Net-(C7-Pad2) -> GND
- D2 pad A: GND -> Net-(D2-PadA)
- D4 pad A: GND -> Net-(D2-PadA)
- R7 pad 1: GND -> Net-(D2-PadA)
- R7 pad 2: Net-(C7-Pad2) -> GND
- RV1 pad 1: Net-(C7-Pad2) -> GND
Routing:
- net Net-(C7-Pad2): track 16.2 -> 0.00 mm
- net Net-(D2-PadA): track 0.00 -> 8.31 mm
Other:
- board text added: "Mini DC-AC Inverter 1.0.2"
- board text removed: "Mini DC-AC Inverter 1.0.1"
Changed lines of the file:
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@@
 		(title "Mini DC-AC Inverter")
 		(date "2025-01-21")
-		(rev "1.0.1")
+		(rev "1.0.2")
 		(comment 1 "Thanks to Ammar for the basics")
 	)
@@
 			(drillshape 0)
 			(scaleselection 1)
-			(outputdirectory "DC-AC-Inverter-EGS-Gerber-1.0.1/")
+			(outputdirectory "DC-AC-Inverter-EGS-Gerber-1.0.2/")
 		)
 	)
@@
 	(net 6 "L")
 	(net 7 "VFB")
-	(net 8 "Net-(C7-Pad2)")
+	(net 8 "Net-(D2-PadA)")
 	(net 9 "Net-(D1-PadC)")
 	(net 10 "Net-(Q2-C)")
@@
 			(layers "*.Cu" "*.Mask")
 			(remove_unused_layers no)
-			(net 1 "GND")
+			(net 8 "Net-(D2-PadA)")
 			(pintype "passive")
 			(solder_mask_margin 0.102)
@@
 			(layers "*.Cu" "*.Mask")
 			(remove_unused_layers no)
-			(net 1 "GND")
+			(net 8 "Net-(D2-PadA)")
 			(pintype "passive")
 			(solder_mask_margin 0.102)
@@
 			(layers "*.Cu" "*.Mask")
 			(remove_unused_layers no)
-			(net 1 "GND")
+			(net 8 "Net-(D2-PadA)")
 			(pintype "passive")
 		)
@@
 			(layers "*.Cu" "*.Mask")
 			(remove_unused_layers no)
-			(net 8 "Net-(C7-Pad2)")
+			(net 1 "GND")
 			(pintype "passive")
 		)
@@
 			)
 		)
-		(property "Value" "22uF 10V"
+		(property "Value" "47uF 10V"
 			(at 1.25 3.75 90)
 			(layer "F.Fab")
@@
 			(layers "*.Cu" "*.Mask")
 			(remove_unused_layers no)
-			(net 8 "Net-(C7-Pad2)")
+			(net 1 "GND")
 			(pinfunction "1")
 			(pintype "passive")
@@
 			(layers "*.Cu" "*.Mask")
 			(remove_unused_layers no)
-			(net 8 "Net-(C7-Pad2)")
+			(net 1 "GND")
 			(pintype "passive")
 		)
@@
 		)
 	)
+	(gr_text "-"
+		(at 101.854 108.7628 0)
+		(layer "F.SilkS")
+		(effects
+			(font
+				(size 1 1)
+				(thickness 0.15)
+			)
+			(justify left bottom)
+		)
+	)
 	(gr_text "stef @ 2025"
 		(at 174.1932 110.236 0)
@@
 		)
 	)
-	(gr_text "Mini DC-AC Inverter 1.0.1"
+	(gr_text "Mini DC-AC Inverter 1.0.2"
 		(at 122.682 93.726 0)
 		(layer "F.SilkS")
@@
 		)
 	)
+	(gr_text "+"
+		(at 111.435 108.815 0)
+		(layer "F.SilkS")
+		(effects
+			(font
+				(size 1 1)
+				(thickness 0.15)
+			)
+			(justify left bottom)
+		)
+	)
 	(gr_text "12V DC IN"
 		(at 104.775 78.359 270)
@@
 	)
 	(segment
-		(start 129.247107 108.165107)
-		(end 128.651 107.569)
-		(width 0.8)
-		(layer "B.Cu")
-		(net 8)
-	)
-	(segment
-		(start 128.651 107.569)
-		(end 128.651 100.562)
-		(width 0.8)
-		(layer "B.Cu")
-		(net 8)
-	)
-	(segment
-		(start 136.1694 107.569)
-		(end 135.573293 108.165107)
-		(width 0.8)
+		(start 147.179507 108.368307)
+		(end 146.3548 107.5436)
+		(width 1)
 		(layer "B.Cu")
 		(net 8)
 	)
 	(segment
-		(start 134.866186 108.458)
-		(end 129.954214 108.458)
-		(width 0.8)
+		(start 150.195 104.6072)
+		(end 150.195 108.6382)
+		(width 1)
 		(layer "B.Cu")
 		(net 8)
 	)
 	(segment
-		(start 128.651 100.562)
-		(end 127.889 99.8)
-		(width 0.8)
-		(layer "B.Cu")
-		(net 8)
-	)
-	(arc
-		(start 135.573293 108.165107)
-		(mid 135.24887 108.38188)
-		(end 134.866186 108.458)
-		(width 0.8)
+		(start 150.218 108.6612)
+		(end 147.886614 108.6612)
+		(width 1)
 		(layer "B.Cu")
 		(net 8)
 	)
 	(arc
-		(start 129.247107 108.165107)
-		(mid 129.57153 108.38188)
-		(end 129.954214 108.458)
-		(width 0.8)
+		(start 147.886614 108.6612)
+		(mid 147.503931 108.58508)
+		(end 147.179507 108.368307)
+		(width 1)
 		(layer "B.Cu")
 		(net 8)
