File: DC-AC-Inverter-EGS-1.0.1/DC-AC-Inverter-EGS.kicad_sch (KiCad schematic)
At the start: 42 parts, among them J1 Fan, J2 EGS002 MODULE, J4 TR/IN, J5 AC/OUT, J6 DC IN, Q1 RM10N100LDV-T, Q2 S8050, Q3 IRF3205, Q4 IRF3205, Q5 IRF3205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

Commit message: Update
Other:
- note added: "Q1 = TSM090N03CP or RM10N100LDV-T"
- note added: "Q2: SS8050DTA or ZTX690BSTZ"
Changed lines of the file:
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@@
 	(title_block
 		(title "Mini DC-AC Inverter")
-		(date "2025-01-21")
+		(date "2025-01-22")
 		(rev "1.0.1")
 		(company "By stef")
@@
 			)
 		)
+	)
+	(text "Q2: SS8050DTA or ZTX690BSTZ"
+		(exclude_from_sim no)
+		(at 80.772 110.744 0)
+		(effects
+			(font
+				(size 1.27 1.27)
+			)
+			(justify left)
+		)
+	)
+	(text "Q1 = TSM090N03CP or RM10N100LDV-T"
+		(exclude_from_sim no)
+		(at 36.322 84.074 0)
+		(effects
+			(font
+				(size 1.27 1.27)
+			)
+		)

Commit message: Update 1.0.2
Connections:
- net GND: now also C7.2, R7.2, RV1.1; no longer D2.A, D4.A, R7.1
- new net: D2.A, D4.A, R7.1
Changed lines of the file:
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@@
 	(title_block
 		(title "Mini DC-AC Inverter")
-		(date "2025-01-22")
-		(rev "1.0.1")
+		(date "2025-01-24")
+		(rev "1.0.2")
 		(company "By stef")
 		(comment 1 "Thanks to Ammar for the basics")
@@
 	(wire
 		(pts
-			(xy 257.81 68.58) (xy 257.81 64.77)
+			(xy 224.79 68.58) (xy 224.79 64.77)
 		)
 		(stroke
@@
 	(symbol
 		(lib_id "power:GND")
-		(at 257.81 68.58 0)
+		(at 224.79 68.58 0)
 		(unit 1)
 		(exclude_from_sim no)
@@
 		(dnp no)
 		(property "Reference" "#PWR022"
-			(at 257.81 74.93 0)
+			(at 224.79 74.93 0)
 			(effects
 				(font
@@
 		)
 		(property "Value" "GND"
-			(at 257.81 72.644 0)
+			(at 224.79 72.644 0)
 			(effects
 				(font
@@
 		)
 		(property "Footprint" ""
-			(at 257.81 68.58 0)
+			(at 224.79 68.58 0)
 			(effects
 				(font
@@
 		)
 		(property "Datasheet" ""
-			(at 257.81 68.58 0)
+			(at 224.79 68.58 0)
 			(effects
 				(font
@@
 		)
 		(property "Description" "Power symbol creates a global label with name \"GND\" , ground"
-			(at 257.81 68.58 0)
+			(at 224.79 68.58 0)
 			(effects
 				(font
